File: 01_DESIGN/server room monitoring/buzzer + led.kicad_sch (KiCad schematic)
At the start: 0 parts

Commit message: Update project files
Parts:
- added BZ1: Buzzer, Buzzer_Beeper:Buzzer_12x9.5RM7.6, symbol Device:Buzzer
- added D10: LED GREEN, LED_SMD:LED_Cree-XHP50_3V_HighDensity, symbol Device:LED
- added D11: LED RED, LED_SMD:LED_Cree-XHP50_3V_HighDensity, symbol Device:LED
- added D9: 1N4148W, Diode_SMD:D_SOD-123, symbol Diode:1N4148W
- added Q3: S8050, Package_TO_SOT_THT:TO-92_Inline, symbol Transistor_BJT:S8050
- added R29, R31, R32: 1k, RES_C_1005x30_L, symbol Device:R
- added R30: 10k, RES_C_1005x30_L, symbol Device:R
Connections:
- new net: D10.2 (A), R31.2
- new net: BZ1.2 (-), D9.2 (A), Q3.3 (C)
- new net: Q3.2 (B), R29.2, R30.2
- new net: D11.2 (A), R32.2
- new net +5V: BZ1.1 (+), D9.1 (K)
- new net BUZZER: R29.1
- new net GND: D10.1 (K), D11.1 (K), Q3.1 (E), R30.1
- new net LED_ALARM: R32.1
- new net LED_STATUS: R31.1
Other:
- note added: "LED_ALARM"
- note added: "LED_STATUS"

Commit message: Update project files
Parts:
- D10, D11: footprint LED_SMD:LED_Cree-XHP50_3V_HighDensity -> LED_SMD:LED_0805_2012Metric
- R29, R30, R31, R32: footprint RES_C_1005x30_L -> Resistor_SMD:R_0805_2012Metric
Changed lines of the file:
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@@
 			)
 		)
-		(property "Footprint" "LED_SMD:LED_Cree-XHP50_3V_HighDensity"
+		(property "Footprint" "LED_SMD:LED_0805_2012Metric"
 			(at 166.37 72.39 0)
 			(hide yes)
@@
 			)
 		)
-		(property "Footprint" "RES_C_1005x30_L"
+		(property "Footprint" "Resistor_SMD:R_0805_2012Metric"
 			(at 46.99 75.438 90)
 			(hide yes)
@@
 			)
 		)
-		(property "Footprint" "LED_SMD:LED_Cree-XHP50_3V_HighDensity"
+		(property "Footprint" "LED_SMD:LED_0805_2012Metric"
 			(at 166.37 101.6 0)
 			(hide yes)
@@
 			)
 		)
-		(property "Footprint" "RES_C_1005x30_L"
+		(property "Footprint" "Resistor_SMD:R_0805_2012Metric"
 			(at 55.118 87.63 90)
 			(hide yes)
@@
 			)
 		)
-		(property "Footprint" "RES_C_1005x30_L"
+		(property "Footprint" "Resistor_SMD:R_0805_2012Metric"
 			(at 148.59 103.378 90)
 			(hide yes)
@@
 			)
 		)
-		(property "Footprint" "RES_C_1005x30_L"
+		(property "Footprint" "Resistor_SMD:R_0805_2012Metric"
 			(at 148.59 74.168 90)
 			(hide yes)
