File: 01_DESIGN/server room monitoring/server room monitoring.kicad_sch (KiCad schematic)
At the start: 0 parts

Commit message: Update project files
Other:
- added sheet ethernet (ethernet.kicad_sch)
- sheet MCU ports: added RS485_DE_~{RE}, RS485_RX, RS485_TX; removed none
- sheet rs485 ports: added RS485_DE_~{RE}, RS485_RX, RS485_TX; removed none
Changed lines of the file:
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@@
 	(generator_version "10.0")
 	(paper "A4")
+	(wire
+		(pts
+			(xy 92.71 107.95) (xy 92.71 106.68)
+		)
+		(stroke
+			(width 0)
+			(type default)
+		)
+	)
+	(wire
+		(pts
+			(xy 83.82 107.95) (xy 92.71 107.95)
+		)
+		(stroke
+			(width 0)
+			(type default)
+		)
+	)
+	(wire
+		(pts
+			(xy 88.9 114.3) (xy 88.9 115.57)
+		)
+		(stroke
+			(width 0)
+			(type default)
+		)
+	)
+	(wire
+		(pts
+			(xy 83.82 125.73) (xy 95.25 125.73)
+		)
+		(stroke
+			(width 0)
+			(type default)
+		)
+	)
+	(wire
+		(pts
+			(xy 83.82 114.3) (xy 88.9 114.3)
+		)
+		(stroke
+			(width 0)
+			(type default)
+		)
+	)
+	(wire
+		(pts
+			(xy 92.71 106.68) (xy 95.25 106.68)
+		)
+		(stroke
+			(width 0)
+			(type default)
+		)
+	)
+	(wire
+		(pts
+			(xy 88.9 115.57) (xy 95.25 115.57)
+		)
+		(stroke
+			(width 0)
+			(type default)
+		)
+	)
 	(sheet
 		(at 226.06 52.07)
@@
 	)
 	(sheet
-		(at 146.05 40.64)
+		(at 134.62 40.64)
+		(size 38.1 40.64)
+		(exclude_from_sim no)
+		(in_bom yes)
+		(on_board yes)
+		(dnp no)
+		(fields_autoplaced yes)
+		(stroke
+			(width 0.1524)
+			(type solid)
+		)
+		(fill
+			(color 0 0 0 0)
+		)
+		(property "Sheetname" "ethernet"
+			(at 134.62 39.9284 0)
+			(show_name no)
+			(do_not_autoplace no)
+			(effects
+				(font
+					(size 1.27 1.27)
+				)
+				(justify left bottom)
+			)
+		)
+		(property "Sheetfile" "ethernet.kicad_sch"
+			(at 134.62 81.8646 0)
+			(show_name no)
+			(do_not_autoplace no)
+			(effects
+				(font
+					(size 1.27 1.27)
+				)
+				(justify left top)
+			)
+		)
+		(instances
+			(project "server room monitoring"
+				(path "/6382e275-058c-4116-9829-3165fddbcf2b"
+					(page "7")
+				)
+			)
+		)
+	)
+	(sheet
+		(at 95.25 97.79)
 		(size 41.91 35.56)
 		(exclude_from_sim no)
@@
 		)
 		(property "Sheetname" "MCU"
-			(at 146.05 39.9284 0)
+			(at 95.25 97.0784 0)
 			(show_name no)
 			(do_not_autoplace no)
@@
 		)
 		(property "Sheetfile" "MCU.kicad_sch"
-			(at 146.05 76.7846 0)
+			(at 95.25 133.9346 0)
 			(show_name no)
 			(do_not_autoplace no)
@@
 				)
 				(justify left top)
+			)
+		)
+		(pin "RS485_RX" bidirectional
+			(at 95.25 115.57 180)
+			(effects
+				(font
+					(size 1.27 1.27)
+				)
+				(justify left)
+			)
+		)
+		(pin "RS485_TX" bidirectional
+			(at 95.25 125.73 180)
+			(effects
+				(font
+					(size 1.27 1.27)
+				)
+				(justify left)
+			)
+		)
+		(pin "RS485_DE_~{RE}" bidirectional
+			(at 95.25 106.68 180)
+			(effects
+				(font
+					(size 1.27 1.27)
+				)
+				(justify left)
 			)
 		)
@@
 			)
 		)
+		(pin "RS485_RX" bidirectional
+			(at 83.82 114.3 0)
+			(effects
+				(font
+					(size 1.27 1.27)
+				)
+				(justify right)
+			)
+		)
+		(pin "RS485_TX" bidirectional
+			(at 83.82 125.73 0)
+			(effects
+				(font
+					(size 1.27 1.27)
+				)
+				(justify right)
+			)
+		)
+		(pin "RS485_DE_~{RE}" bidirectional
+			(at 83.82 107.95 0)
+			(effects
+				(font
+					(size 1.27 1.27)
+				)
+				(justify right)
+			)
+		)

Commit message: Update project files
Other:
- sheet MCU ports: added BUZZER, ETH_CS, ETH_INT, ETH_MISO, ETH_MOSI, ETH_RST, ETH_SCK, LED_ALARM, LED_STATUS; removed none
- sheet buzzer + led ports: added BUZZER, LED_ALARM, LED_STATUS; removed none
- sheet ethernet ports: added ETH_CS, ETH_INT, ETH_MISO, ETH_MOSI, ETH_RST, ETH_SCK; removed none
