File: 01_DESIGN/server room monitoring/MCU.kicad_sch (KiCad schematic)
At the start: 10 parts, among them J2 HEADER 4x1, SW1 SW_Push, SW2 SW_Push, U3 ESP32-WROOM-32E

Commit message: Update project files
Parts:
- removed C7: 0.1uF, symbol Device:C
- added J5: Conn_01x07_Pin, Connector_PinHeader_2.54mm:PinHeader_1x07_P2.54mm_Vertical, symbol Connector:Conn_01x07_Pin
- added J7: USB_C_Receptacle_USB2.0_16P, Connector_USB:USB3_A_Molex_48393-001, symbol Connector:USB_C_Receptacle_USB2.0_16P
- C5: value 22uF -> 10uF
Connections:
- net 4G_RX: now also J5.4 (Pin_4)
- net 4G_TX: now also J5.3 (Pin_3)
- net GND: now also J5.2 (Pin_2)
- net IO27: now reaches U3.12 (IO27)
- net IO27: now also J5.5 (Pin_5)
- net ETH_RST: now reaches U3.13 (IO14)
- net ETH_CS: now reaches U3.29 (IO5)
- net ETH_SCK: now reaches U3.30 (IO18)
- net ETH_MISO: now reaches U3.31 (IO19)
- net ETH_MOSI: now reaches U3.37 (IO23)
- net ETH_INT: now reaches U3.6 (IO34)
- net RS485_DE_RE renamed RS485_DE_~{RE}
- new net: J7.A1 (GND), J7.A12 (GND), J7.B1 (GND), J7.B12 (GND)
- new net: J7.A4 (VBUS), J7.A9 (VBUS), J7.B4 (VBUS), J7.B9 (VBUS)
- new net +5V: J5.1 (Pin_1)
- no-connect marks 16 -> 11
Other:
- note added: "CONNECT MODULE 4G"
- note added: "ESP 32 WROOM 32E N4"
- moved on the sheet: C5, C6, C8, J2, R3, R4, SW1, SW2, U3

Commit message: Update project files
Parts:
- removed J2: HEADER 4x1, symbol AL:Header 4x1
- removed J7: USB_C_Receptacle_USB2.0_16P, Connector_USB:USB3_A_Molex_48393-001, symbol Connector:USB_C_Receptacle_USB2.0_16P
- added C29, C7: 0.1uF, symbol Device:C
- added D5: SS34, Diode_SMD:D_SMA, symbol Diode:SS34
- added J7: 2171790001, 2171790001:2171790001_MOL, symbol 2171790001:2171790001
- added Q1, Q2: S8050, Package_TO_SOT_THT:TO-92_Inline, symbol Transistor_BJT:S8050
- added R24, R25: 5.1k, symbol Device:R
- added R26, R27: 10k, symbol Device:R
- added U6: CH340C, Package_SO:SOIC-16_3.9x9.9mm_P1.27mm, symbol Interface_USB:CH340C
- added U7: USBLC6-2SC6, Package_TO_SOT_SMD:SOT-23-6, symbol Power_Protection:USBLC6-2SC6
Connections:
- net 4G_RX: now also U3.28 (IO17); no longer U3.11 (IO26)
- net 4G_TX: now also U3.27 (IO16); no longer U3.10 (IO25)
- net BUZZER: now also U3.10 (IO25); no longer U3.8 (IO32)
- net GND: now also C7.1, J7.A1/B12 (GND_2), J7.B1/A12 (GND), R24.1, R25.1, U6.1 (GND), U7.2 (GND)
- net RS485_DE_~{RE}: now also U3.16 (IO13); no longer U3.26 (IO4)
- net RS485_RX: now also U3.36 (IO22); no longer U3.27 (IO16)
- net RS485_TX: now also U3.33 (IO21); no longer U3.28 (IO17)
- net UART0_RX: now also U6.2 (TXD)
- net UART0_TX: now also U6.3 (RXD)
- net ESP_EN: now reaches C8.2, R3.1, SW1.2, U3.3 (EN)
- net ESP_EN: now also Q1.3 (C)
- net 4G_NET: now reaches J5.6 (Pin_6)
- net 4G_NET: now also U3.7 (IO35)
- net 4G_DTR: now reaches J5.7 (Pin_7)
- net 4G_DTR: now also U3.8 (IO32)
- net ESP_BOOT: now reaches R4.2, SW2.1, U3.25 (IO0)
- net ESP_BOOT: now also Q2.3 (C)
- net IO27 renamed 4G_EN
- net 4G_EN: now also U3.26 (IO4); no longer U3.12 (IO27)
- net SENSOR_DATA: no longer names the net of U3.9 (IO33)
- new net: Q2.1 (E), R26.2, U6.14 (~{RTS})
- new net: Q2.2 (B), R27.1
- new net: J7.A5 (CC1), R24.2
- new net: Q1.1 (E), R27.2, U6.13 (~{DTR})
- new net: C7.2, U6.4 (V3)
- new net: C29.1, U6.16 (VCC)
- new net: U6.5 (UD+), U7.6 (I/O1)
- new net: U6.6 (UD-), U7.4 (I/O2)
- new net: Q1.2 (B), R26.1
- new net: J7.A6 (DP1), J7.B6 (DP2), U7.1 (I/O1)
- new net: J7.A7 (DN1), J7.B7 (DN2), U7.3 (I/O2)
- new net: J7.B5 (CC2), R25.2
- new net 5V_USB: C29.2, D5.1 (K)
- new net LED_ALARM: U3.12 (IO27)
- new net LED_STATUS: U3.11 (IO26)
- new net VBUS: D5.2 (A), J7.A4/B9 (VBUS_2), J7.B4/A9 (VBUS), U7.5 (VBUS)
- no-connect marks 11 -> 12
Other:
- note added: "USBC 2.0"
- moved on the sheet: C5, C6, C8, J5, R3, R4, SW1, SW2, U3

Commit message: Update project files
Parts:
- C29, C5, C6, C7, C8: footprint (none) -> Capacitor_SMD:C_0805_2012Metric
- Q1, Q2: footprint Package_TO_SOT_THT:TO-92_Inline -> Package_TO_SOT_SMD:SOT-23
- R24, R25, R26, R27, R3, R4: footprint (none) -> Resistor_SMD:R_0805_2012Metric
- SW1, SW2: footprint (none) -> Button_Switch_SMD:SW_SPST_PTS645Sx43SMTR92
Connections:
- net VBUS is gone; now on net 5V_USB: D5.2 (A), J7.A4/B9 (VBUS_2), J7.B4/A9 (VBUS), U7.5 (VBUS)
- no-connect marks 12 -> 13
Other:
- moved on the sheet: D5
Changed lines of the file:
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@@
 	)
 	(junction
+		(at 176.53 46.99)
+		(diameter 0)
+		(color 0 0 0 0)
+	)
+	(junction
 		(at 62.23 45.72)
 		(diameter 0)
@@
 	)
 	(junction
+		(at 271.78 66.04)
+		(diameter 0)
+		(color 0 0 0 0)
+	)
+	(junction
 		(at 257.81 66.04)
 		(diameter 0)
@@
 	)
 	(no_connect
+		(at 184.15 58.42)
+	)
+	(no_connect
 		(at 163.83 71.12)
 	)
@@
 	(wire
 		(pts
+			(xy 257.81 59.69) (xy 257.81 63.5)
+		)
+		(stroke
+			(width 0)
+			(type default)
+		)
+	)
+	(wire
+		(pts
 			(xy 88.9 74.93) (xy 88.9 63.5)
 		)
@@
 	(wire
 		(pts
-			(xy 264.16 66.04) (xy 257.81 66.04)
+			(xy 262.89 66.04) (xy 257.81 66.04)
 		)
 		(stroke
@@
 	(wire
 		(pts
+			(xy 271.78 66.04) (xy 270.51 66.04)
+		)
+		(stroke
+			(width 0)
+			(type default)
+		)
+	)
+	(wire
+		(pts
 			(xy 185.42 93.98) (xy 185.42 66.04)
 		)
@@
 			)
 		)
-		(property "Footprint" "Package_TO_SOT_THT:TO-92_Inline"
+		(property "Footprint" "Package_TO_SOT_SMD:SOT-23"
 			(at 144.145 102.87 0)
 			(hide yes)
@@
 	(symbol
 		(lib_id "power:+5V")
-		(at 257.81 63.5 0)
+		(at 257.81 59.69 0)
 		(unit 1)
 		(body_style 1)
@@
 		(in_pos_files yes)
 		(dnp no)
-		(fields_autoplaced yes)
 		(property "Reference" "#PWR081"
-			(at 257.81 67.31 0)
+			(at 257.81 63.5 0)
 			(hide yes)
 			(show_name no)
@@
 			)
 		)
-		(property "Value" "VBUS"
-			(at 257.81 58.42 0)
+		(property "Value" "5V_USB"
+			(at 255.27 55.118 0)
 			(show_name no)
 			(do_not_autoplace no)
@@
 					(size 1.27 1.27)
 				)
+				(justify left)
 			)
 		)
 		(property "Footprint" ""
-			(at 257.81 63.5 0)
+			(at 257.81 59.69 0)
 			(hide yes)
 			(show_name no)
@@
 		)
 		(property "Datasheet" ""
-			(at 257.81 63.5 0)
+			(at 257.81 59.69 0)
 			(hide yes)
 			(show_name no)
@@
 		)
 		(property "Description" "Power symbol creates a global label with name \"+5V\""
-			(at 257.81 63.5 0)
+			(at 257.81 59.69 0)
 			(hide yes)
 			(show_name no)
@@
 			)
 		)
-		(property "Footprint" ""
+		(property "Footprint" "Resistor_SMD:R_0805_2012Metric"
 			(at 200.66 60.198 90)
 			(hide yes)
@@
 			)
 		)
-		(property "Footprint" ""
+		(property "Footprint" "Resistor_SMD:R_0805_2012Metric"
 			(at 55.118 62.23 90)
 			(hide yes)
@@
 			)
 		)
-		(property "Footprint" ""
+		(property "Footprint" "Resistor_SMD:R_0805_2012Metric"
 			(at 144.018 85.09 90)
 			(hide yes)
@@
 			)
 		)
-		(property "Footprint" ""
+		(property "Footprint" "Button_Switch_SMD:SW_SPST_PTS645Sx43SMTR92"
 			(at 97.79 69.85 0)
 			(hide yes)
@@
 		(in_pos_files yes)
 		(dnp no)
-		(fields_autoplaced yes)
 		(property "Reference" "#PWR083"
 			(at 195.58 86.36 0)
@@
 			)
 		)
-		(property "Value" "VBUS"
-			(at 195.58 77.47 0)
+		(property "Value" "5V_USB"
+			(at 192.532 78.486 0)
 			(show_name no)
 			(do_not_autoplace no)
@@
 					(size 1.27 1.27)
 				)
+				(justify left)
 			)
 		)
@@
 			)
 		)
-		(property "Footprint" ""
+		(property "Footprint" "Capacitor_SMD:C_0805_2012Metric"
 			(at 168.91 46.0248 0)
 			(hide yes)
@@
 			)
 		)
-		(property "Footprint" ""
+		(property "Footprint" "Capacitor_SMD:C_0805_2012Metric"
 			(at 26.3652 53.34 0)
 			(hide yes)
@@
 			)
 		)
-		(property "Footprint" "Package_TO_SOT_THT:TO-92_Inline"
+		(property "Footprint" "Package_TO_SOT_SMD:SOT-23"
 			(at 156.845 102.87 0)
 			(hide yes)
@@
 			)
 		)
-		(property "Footprint" ""
+		(property "Footprint" "Button_Switch_SMD:SW_SPST_PTS645Sx43SMTR92"
 			(at 26.67 69.85 0)
 			(hide yes)
@@
 	(symbol
 		(lib_id "Diode:SS34")
-		(at 267.97 66.04 180)
+		(at 266.7 66.04 180)
 		(unit 1)
 		(body_style 1)
@@
 		(dnp no)
 		(property "Reference" "D5"
-			(at 267.97 68.58 0)
+			(at 266.7 68.58 0)
 			(show_name no)
 			(do_not_autoplace no)
@@
 		)
 		(property "Value" "SS34"
-			(at 268.732 63.754 0)
+			(at 267.462 63.754 0)
 			(show_name no)
 			(do_not_autoplace no)
@@
 		)
 		(property "Footprint" "Diode_SMD:D_SMA"
-			(at 267.97 61.595 0)
+			(at 266.7 61.595 0)
 			(hide yes)
 			(show_name no)
@@
 		)
 		(property "Datasheet" "https://www.vishay.com/docs/88751/ss32.pdf"
-			(at 267.97 66.04 0)
+			(at 266.7 66.04 0)
 			(hide yes)
 			(show_name no)
@@
 		)
 		(property "Description" "40V 3A Schottky Diode, SMA"
-			(at 267.97 66.04 0)
+			(at 266.7 66.04 0)
 			(hide yes)
 			(show_name no)
@@
 	)
 	(symbol
+		(lib_id "power:PWR_FLAG")
+		(at 271.78 66.04 180)
+		(unit 1)
+		(body_style 1)
+		(exclude_from_sim no)
+		(in_bom yes)
+		(on_board yes)
+		(in_pos_files yes)
+		(dnp no)
+		(fields_autoplaced yes)
+		(property "Reference" "#FLG07"
+			(at 271.78 67.945 0)
+			(hide yes)
+			(show_name no)
+			(do_not_autoplace no)
+			(effects
+				(font
+					(size 1.27 1.27)
+				)
+			)
+		)
+		(property "Value" "PWR_FLAG"
+			(at 271.78 71.12 0)
+			(show_name no)
+			(do_not_autoplace no)
+			(effects
+				(font
+					(size 1.27 1.27)
+				)
+			)
+		)
+		(property "Footprint" ""
+			(at 271.78 66.04 0)
+			(hide yes)
+			(show_name no)
+			(do_not_autoplace no)
+			(effects
+				(font
+					(size 1.27 1.27)
+				)
+			)
+		)
+		(property "Datasheet" ""
+			(at 271.78 66.04 0)
+			(hide yes)
+			(show_name no)
+			(do_not_autoplace no)
+			(effects
+				(font
+					(size 1.27 1.27)
+				)
+			)
+		)
+		(property "Description" "Special symbol for telling ERC where power comes from"
+			(at 271.78 66.04 0)
+			(hide yes)
+			(show_name no)
+			(do_not_autoplace no)
+			(effects
+				(font
+					(size 1.27 1.27)
+				)
+			)
+		)
+		(pin "1"
+		)
+		(instances
+			(project "server room monitoring"
+				(path "/6382e275-058c-4116-9829-3165fddbcf2b/234b9206-bcdf-4a8c-be0b-cbb776d074a9"
+					(reference "#FLG07")
+					(unit 1)
+				)
+			)
+		)
+	)
+	(symbol
 		(lib_id "Power_Protection:USBLC6-2SC6")
 		(at 195.58 91.44 0)
@@
 			)
 		)
-		(property "Footprint" ""
+		(property "Footprint" "Capacitor_SMD:C_0805_2012Metric"
 			(at 30.48 67.6148 0)
 			(hide yes)
@@
 			)
 		)
-		(property "Footprint" ""
+		(property "Footprint" "Capacitor_SMD:C_0805_2012Metric"
 			(at 37.7952 53.34 0)
 			(hide yes)
@@
 			)
 		)
-		(property "Footprint" ""
+		(property "Footprint" "Resistor_SMD:R_0805_2012Metric"
 			(at 160.528 85.09 90)
 			(hide yes)
@@
 	)
 	(symbol
+		(lib_id "power:PWR_FLAG")
+		(at 176.53 46.99 0)
+		(unit 1)
+		(body_style 1)
+		(exclude_from_sim no)
+		(in_bom yes)
+		(on_board yes)
+		(in_pos_files yes)
+		(dnp no)
+		(fields_autoplaced yes)
+		(property "Reference" "#FLG09"
+			(at 176.53 45.085 0)
+			(hide yes)
+			(show_name no)
+			(do_not_autoplace no)
+			(effects
+				(font
+					(size 1.27 1.27)
+				)
+			)
+		)
+		(property "Value" "PWR_FLAG"
+			(at 176.53 41.91 0)
+			(show_name no)
+			(do_not_autoplace no)
+			(effects
+				(font
+					(size 1.27 1.27)
+				)
+			)
+		)
+		(property "Footprint" ""
+			(at 176.53 46.99 0)
+			(hide yes)
+			(show_name no)
+			(do_not_autoplace no)
+			(effects
+				(font
+					(size 1.27 1.27)
+				)
+			)
+		)
+		(property "Datasheet" ""
+			(at 176.53 46.99 0)
+			(hide yes)
+			(show_name no)
+			(do_not_autoplace no)
+			(effects
+				(font
+					(size 1.27 1.27)
+				)
+			)
+		)
+		(property "Description" "Special symbol for telling ERC where power comes from"
+			(at 176.53 46.99 0)
+			(hide yes)
+			(show_name no)
+			(do_not_autoplace no)
+			(effects
+				(font
+					(size 1.27 1.27)
+				)
+			)
+		)
+		(pin "1"
+		)
+		(instances
+			(project "server room monitoring"
+				(path "/6382e275-058c-4116-9829-3165fddbcf2b/234b9206-bcdf-4a8c-be0b-cbb776d074a9"
+					(reference "#FLG09")
+					(unit 1)
+				)
+			)
+		)
+	)
+	(symbol
 		(lib_id "power:GND")
 		(at 250.19 58.42 180)
@@
 			)
 		)
-		(property "Footprint" ""
+		(property "Footprint" "Capacitor_SMD:C_0805_2012Metric"
 			(at 187.96 46.0248 0)
 			(hide yes)
@@
 			)
 		)
-		(property "Footprint" ""
+		(property "Footprint" "Resistor_SMD:R_0805_2012Metric"
 			(at 87.122 59.69 90)
 			(hide yes)
@@
 			)
 		)
-		(property "Footprint" ""
+		(property "Footprint" "Resistor_SMD:R_0805_2012Metric"
 			(at 200.66 62.738 90)
 			(hide yes)

Commit message: Update project files
Parts:
- removed C5: 10uF, Capacitor_SMD:C_0805_2012Metric, symbol Device:C_Polarized
- added C41, C5: 10uF, Capacitor_SMD:C_0805_2012Metric, symbol Device:C
- added R43, R44: 470R, Resistor_SMD:R_0805_2012Metric, symbol Device:R
Connections:
- net +3.3V: now also C5.1
- net 5V_USB: now also C41.2
- net ESP_BOOT: now also Q1.3 (C); no longer Q2.3 (C)
- net ESP_EN: now also Q2.3 (C); no longer Q1.3 (C)
- net GND: now also C5.2
- net UART0_RX: now also R43.1; no longer U6.2 (TXD)
- net UART0_TX: now also R44.1; no longer U6.3 (RXD)
- net at C29.1, U6.16 (VCC): now also C41.1
- new net: R43.2, U6.2 (TXD)
- new net: R44.2, U6.3 (RXD)
Other:
- moved on the sheet: C29
