File: 01_DESIGN/server room monitoring/power.kicad_sch (KiCad schematic)
At the start: 17 parts, among them J1 Screw_Terminal_01x02, U1 LM2596S-5, U2 LM1117MP-3.3

Commit message: Update project files
Parts:
- removed C3: 470uF, symbol Device:C
- added C3: 470uF, Package_DIP:DIP-24_W7.62mm, symbol Device:C_Polarized
- added C30, C32, C33: 0.1uF, symbol Device:C
- added C31: 10uF, symbol Device:C
- added D6: SMAJ28A, Diode_SMD:D_SMA, symbol Diode:SMAJ28A
- added D7: SS34, Diode_SMD:D_SMA, symbol Diode:SS34
- added D8: LED, symbol Device:LED
- added F1: MF-MSMF250_16X-2, MF-MSMF250_16X-2:FUSER_MF-MSMF250_16X-2, symbol MF-MSMF250_16X-2:MF-MSMF250_16X-2
- added R28: 1k, symbol Device:R
- C1: value 10uF -> 0.1uF
Connections:
- net +12V: now also J1.1 (Pin_1), F1.1; no longer J1.2 (Pin_2), U1.1 (VIN)
- net +3.3V: now also C32.1
- net +5V: now also C31.1, C33.1
- net GND: now also J1.2 (Pin_2), C3.2, C30.2, C31.2, C32.2, C33.2, D6.2 (A2), D7.2 (A), D8.1 (K); no longer D1.2 (A), J1.1 (Pin_1)
- net at L1.2, U1.2 (OUT): now also D7.1 (K); no longer D1.1 (K)
- new net: D1.2 (A), F1.2
- new net: D8.2 (A), R28.2
- new net 12V_PROT: C3.1, C30.1, D1.1 (K), D6.1 (A1), R28.1, U1.1 (VIN)
Other:
- note added: "POWER INPUT"
- moved on the sheet: C1, C2, C4, D1, D2, D3, H1, H2, H3, H4, J1, L1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

Commit message: Update project files
Parts:
- added TP3, TP4, TP5, TP6: TestPoint, TestPoint:TestPoint_Pad_D1.0mm, symbol Connector:TestPoint
- C1, C2, C30, C31, C32, C33: footprint (none) -> Capacitor_SMD:C_0805_2012Metric
- C3: footprint Package_DIP:DIP-24_W7.62mm -> Capacitor_SMD:CP_Elec_10x10.5
- C4: footprint (none) -> Capacitor_SMD:CP_Elec_8x10.5
- D1, D7: footprint Diode_SMD:D_SMA -> Diode_SMD:D_SMC
- D2, D3, D8: footprint (none) -> LED_SMD:LED_0805_2012Metric
- H1, H2, H3, H4: now in the parts list
- L1: footprint (none) -> Inductor_SMD:L_12x12mm_H8mm
- R1, R2, R28: footprint (none) -> Resistor_SMD:R_0805_2012Metric
Connections:
- net +3.3V: now also TP5.1
- net +5V: now also TP4.1
- net 12V_PROT: now also TP3.1; no longer D6.1 (A1)
- net GND: now also TP6.1
- net at D1.2 (A), F1.2: now also D6.1 (A1)
Other:
- moved on the sheet: D1, D6

Commit message: Update project files
Parts:
- removed C2: 10uF, Capacitor_SMD:C_0805_2012Metric, symbol Device:C
- removed D6: SMAJ28A, Diode_SMD:D_SMA, symbol Diode:SMAJ28A
- removed F1: MF-MSMF250_16X-2, MF-MSMF250_16X-2:FUSER_MF-MSMF250_16X-2, symbol MF-MSMF250_16X-2:MF-MSMF250_16X-2
- added C2: 10uF, Capacitor_Tantalum_SMD:CP_EIA-3216-18_Kemet-A, symbol Device:C_Polarized
- added D6: SMAJ14A, Diode_SMD:D_SMA, symbol Diode:SMAJ14A
- added F1: MF-MSMF260-2, MF-MSMF260-2:FUSE_MF-MSMF260-2, symbol MF-MSMF260-2:MF-MSMF260-2
- C3: value 470uF -> 120uF
- C4: value 220uF -> 330uF
- L1: value 68uH -> 33uH
Connections:
- net +12V: now also F1.1
- net +3.3V: now also C2.1
- net GND: now also C2.2, D6.2 (A2)
- net at D1.2 (A): now also D6.1 (A1), F1.2
